Commit message: demo

File: iqr_kobuki_description/urdf/iqr_kobuki_robot.urdf.xacro (robot description, xacro)
@@ -1,15 +1,39 @@
 <?xml version="1.0"?>
-<robot xmlns:xacro="http://www.ros.org/wiki/xacro" name="iqr_4b_robot">
+<robot xmlns:xacro="http://www.ros.org/wiki/xacro" name="iqr_kobuki_robot">
   <xacro:include filename="$(find iqr_kobuki_description)/urdf/zed.xacro"/>
   <xacro:include filename="$(find iqr_kobuki_description)/urdf/vlp16.xacro"/>
   <xacro:include filename="$(find kobuki_description)/urdf/kobuki.urdf.xacro" />
   <kobuki/>
-    <!-- VLP-16 lidar -->
+  <!-- support -->
+  <link name="support_link">
+      <visual>
+        <origin xyz="0 0 0" rpy="0 0 0"/>
+        <geometry>
+          <mesh filename="package://iqr_kobuki_description/meshes/turtlebot_support.stl"/>
+        </geometry>
+        <material name="">
+          <color rgba="0.3 0.3 0.3 1"/>
+        </material>
+      </visual>
+  </link>
+  <joint name="support_link_joint" type="fixed">
+      <origin xyz="0 0 0" rpy="0 0 0" />
+      <parent link="base_footprint"/>
+      <child link="support_link"/>
+  </joint>
+  <!-- JY901 -->
+  <link name="imu_link"/>
+  <joint name="imu_link_joint" type="fixed">
+      <origin xyz="0 0 0.123" rpy="0 0 0" />
+      <parent link="base_footprint"/>
+      <child link="imu_link"/>
+  </joint>
+  <!-- VLP-16 lidar -->
   <xacro:vlp16 package="iqr_kobuki_description" parent="base_footprint">
-    <origin xyz="-0.005 0 0.528" rpy="0 0 0" />
+    <origin xyz="-0.005 0 0.3438" rpy="0 0 0" />
   </xacro:vlp16>
   <!-- ZED Camera -->
   <xacro:zed package="iqr_kobuki_description" parent="base_footprint">
-    <origin xyz="0.27193 0 -0.06943" rpy="0 0 0" />
+    <origin xyz="0.119 0 0.278" rpy="0 0 0" />
   </xacro:zed>
   </robot>

File: iqr_kobuki_description/urdf/vlp16.xacro (robot description, xacro)
@@ -19,10 +19,10 @@
       <child link="${prefix}_link"/>
     </joint>
-<!--     <link name="velodyne"/>
+  <link name="velodyne"/>
     <joint name="velodyne_link_joint" type="fixed">
       <origin xyz="0 0 0.040" rpy="0 0 0" />
       <parent link="${prefix}_link"/>
       <child link="velodyne"/>
-    </joint> -->
+    </joint>
   </xacro:macro>
 </robot>

File: iqr_kobuki_description/urdf/zed.xacro (robot description, xacro)
@@ -19,4 +19,47 @@
       <child link="${prefix}_link"/>
     </joint>
+<!-- Camera Center -->
+    <joint name="zed_camera_center_joint" type="fixed">
+        <parent link="${prefix}_link"/>
+        <child link="zed_camera_center"/>
+        <origin xyz="0 0 0" rpy="0 0 0" />
+    </joint>
+    <link name="zed_camera_center">
+        <visual>
+            <origin xyz="0 0 0" rpy="0 0 0"/>
+            <geometry>
+                <mesh filename="package://zed_wrapper/urdf/models/ZED.stl" />
+            </geometry>
+            <material name="light_grey">
+                <color rgba="0.8 0.8 0.8 0.8"/>
+            </material>
+        </visual>
+    </link>
+<!-- Left Camera -->
+    <joint name="zed_left_camera_joint" type="fixed">
+        <parent link="zed_camera_center"/>
+        <child link="zed_left_camera_frame"/>
+        <origin xyz="0 0.06 0" rpy="0 0 0" />
+    </joint>
+    <link name="zed_left_camera_frame" />
+    <joint name="zed_left_camera_optical_joint" type="fixed">
+        <origin xyz="0 0 0" rpy="-1.57079632679 0.0 -1.57079632679"/>
+        <parent link="zed_left_camera_frame"/>
+        <child link="zed_left_camera_optical_frame"/>
+    </joint>
+    <link name="zed_left_camera_optical_frame"/>
+<!-- Right Camera -->
+    <joint name="zed_right_camera_joint" type="fixed">
+        <parent link="zed_camera_center"/>
+        <child link="zed_right_camera_frame"/>
+        <origin xyz="0 -0.06 0" rpy="0 0 0" />
+    </joint>
+    <link name="zed_right_camera_frame" />
+    <joint name="zed_right_camera_optical_joint" type="fixed">
+        <origin xyz="0 0 0" rpy="-1.57079632679 0.0 -1.57079632679"/>
+        <parent link="zed_right_camera_frame"/>
+        <child link="zed_right_camera_optical_frame"/>
+    </joint>
+    <link name="zed_right_camera_optical_frame"/>
   </xacro:macro>
 </robot>
